File: ft232r-eval.kicad_pcb (KiCad board)
At the start: 2 copper layers, 25 x 51 mm, 15 parts, among them J1 USB_A, J2 FTDI, J3 JST, SW1 VIO_SEL, U1 FT232RL

Commit message: License under CC BY 4.0
Other:
- board text added: "FT232R Evaluation Board v2 C. Keller 2021-04-05 https://github.com/k0swe/ft232r-eval"
- board text removed: "FT232R Evaluation Board v2 C. Keller 2021-04-05"

Commit message: Small updates
Other:
- net class Data added: clearance 0.2, trace_width 0.2, via_dia 0.8, via_drill 0.4
- board text added: "FT232R Evaluation Board v2 C. Keller 2021-04-18 https://github.com/k0swe/ft232r-eval"
- board text removed: "3V3 VCCIO 5V"
- board text removed: "CTS"
- board text removed: "DTR"
- board text removed: "FT232R Evaluation Board v2 C. Keller 2021-04-05 https://github.com/k0swe/ft232r-eval"
- board text removed: "GND"
- board text removed: "RX"
- board text removed: "TX"
- board text removed: "VCCIO"

Commit message: Add OSHW logo
Parts:
- added LOGO1: Logo_Open_Hardware_Small, Symbol:OSHW-Logo2_9.8x8mm_SilkScreen, B.Cu at (151.0, 82.0)
