File: ft232r-eval.sch (KiCad schematic (older format))
At the start: 15 parts, among them J1 USB_A, J2 FTDI, J3 JST, SW1 VIO_SEL, U1 FT232RL

Commit message: Fix FTDI header footprint
Parts:
- J2: footprint Connector_PinSocket_2.54mm:PinSocket_1x06_P2.54mm_Vertical_SMD_Pin1Left -> Connector_PinSocket_2.54mm:PinSocket_1x06_P2.54mm_Vertical
Changed lines of the file:
@@
 F 0 "J2" H 7980 2992 50 0000 L CNN
 F 1 "FTDI" H 7980 2901 50 0000 L CNN
-F 2 "Connector_PinSocket_2.54mm:PinSocket_1x06_P2.54mm_Vertical_SMD_Pin1Left" H 7900 3000 50 0001 C CNN
+F 2 "Connector_PinSocket_2.54mm:PinSocket_1x06_P2.54mm_Vertical" H 7900 3000 50 0001 C CNN
 F 3 "https://www.mouser.com/datasheet/2/1/ts0815-31700.pdf" H 7900 3000 50 0001 C CNN
 F 4 "0.8" H 7980 3092 50 0001 C CNN "Price"

Commit message: Add OSHW logo
Parts:
- added LOGO1: Logo_Open_Hardware_Small, Symbol:OSHW-Logo2_9.8x8mm_SilkScreen, symbol Graphic:Logo_Open_Hardware_Small
Changed lines of the file:
@@
 Connection ~ 8650 4550
 Connection ~ 6200 2150
+$Comp
+L Graphic:Logo_Open_Hardware_Small LOGO1
+U 1 1 6086E6E2
+P 10900 6850
+F 0 "LOGO1" H 10900 7125 50  0001 C CNN
+F 1 "Logo_Open_Hardware_Small" H 10900 6625 50  0001 C CNN
+F 2 "Symbol:OSHW-Logo2_9.8x8mm_SilkScreen" H 10900 6850 50  0001 C CNN
+F 3 "~" H 10900 6850 50  0001 C CNN
+	1    10900 6850
+	1    0    0    -1
+$EndComp
 $EndSCHEMATC
